File: bdm-reverb.kicad_sch (KiCad schematic)
At the start: 0 parts

Commit message: iroiro
Parts:
- added C1, C12, C14, C15, C16, C27, C29, C3, C31, C33, C34: 0.1u, symbol Device:C
- added C10, C9: 2.2n, symbol Device:C
- added C11, C13: 4.7u, symbol Device:C
- added C17, C18, C2, C35, C36, C4, C7, C8: 10u, symbol Device:C
- added C19: C, symbol Device:C
- added C20: 100u, symbol Device:C
- added C21: 220u, symbol Device:C
- added C22, C25: 100n, symbol Device:C
- added C23, C28, C30, C32, C5, C6: 1u, symbol Device:C
- added C24: 22u, symbol Device:C
- added C26: 220n, symbol Device:C
- added D1, D2, D3, D4: 1N5819, Diode_THT:D_DO-41_SOD81_P10.16mm_Horizontal, symbol Diode:1N5819
- added D5, D6: 1N4007, Diode_THT:D_DO-41_SOD81_P10.16mm_Horizontal, symbol Diode:1N4007
- added D7: LED, symbol Device:LED
- added FB1: FerriteBead, symbol Device:FerriteBead
- added J1: input jack (line), symbol Connector_Audio:AudioJack2
- added J2: input jack (piezo), symbol Connector_Audio:AudioJack2
- added J3: output jack (line), symbol Connector_Audio:AudioJack2
- added J4: output jack (spk), symbol Connector_Audio:AudioJack2
- added J5: Conn_02x08_Top_Bottom, symbol Connector_Generic:Conn_02x08_Top_Bottom
- added R1, R2: 150, symbol Device:R
- added R10, R17, R3, R4, R5, R6, R7, R8, R9: 10k, symbol Device:R
- added R11: 100k, symbol Device:R
- added R12: 22k, symbol Device:R
- added R13: 680, symbol Device:R
- added R14: 1, symbol Device:R
- added R15: 13k, symbol Device:R
- added R16: 5k, symbol Device:R
- added R18: 2, symbol Device:R
- added RV1, RV2, RV3, RV4, RV5: R_Potentiometer, symbol Device:R_Potentiometer
- added SW1: SW_DPST, symbol Switch:SW_DPST
- added U1: Teensy4.0, Teensy:Teensy40, symbol teensy:Teensy4.0
- added U2, U3, U5: TL072, symbol Amplifier_Operational:TL072
- added U4: TDA2030, Package_TO_SOT_THT:TO-220-5_P3.4x3.7mm_StaggerOdd_Lead3.8mm_Vertical, symbol Amplifier_Audio:TDA2030
- added VM4220M1: ~, symbol V4220M:V4220M
Connections:
- new net: R4.2, R7.1, U3.6 (-)
- new net: R7.2, VM4220M1.26 (LOUT-)
- new net: D5.1 (K), D6.2 (A), J4.T, R14.1, R15.2, U4.4
- new net: C26.1, R14.2
- new net: C21.1, C25.1, D6.1 (K), SW1.3, U4.5 (+Vs)
- new net: C23.1, R12.1, U4.1 (+)
- new net: R13.1, U4.2 (-)
- new net: C20.1, C22.1, D5.2 (A), SW1.1, U4.3 (-Vs)
- new net: RV1.1, U2.1, U2.2 (-)
- new net: C7.1, RV1.2
- new net: C8.2, R2.1
- new net: C10.1, R2.2, VM4220M1.20 (LIN+)
- new net: C31.1, C32.1, R18.2, VM4220M1.6 (VD)
- new net: C5.2, U2.3 (+)
- new net: C13.1, C14.1, VM4220M1.19 (LIN-)
- new net: C11.1, C12.1, VM4220M1.16 (RIN-)
- new net: C19.1, J3.T, R11.2
- new net: C7.2, R1.1
- new net: C9.1, R1.2, VM4220M1.17 (RIN+)
- new net: R6.2, R8.2, U3.3 (+)
- new net: R8.1, VM4220M1.24 (ROUT+)
- new net: C27.1, C28.1, R17.1, RV5.3, U1.31 (3V3), VM4220M1.13 (VL)
- new net: R10.2, VM4220M1.23 (ROUT-)
- new net: R9.1, VM4220M1.25 (LOUT+)
- new net: R17.2, VM4220M1.27 (RSTN)
- new net: U1.30 (23_A9_CRX1_MCLK1), VM4220M1.3 (XTI)
- new net: U1.27 (20_A6_TX5_LRCLK1), VM4220M1.4 (LRCK)
- new net: U1.28 (21_A7_RX5_BCLK1), VM4220M1.5 (SLCK)
- new net: U1.10 (8_TX2_IN1), VM4220M1.8 (DOUT)
- new net: U1.9 (7_RX2_OUT1A), VM4220M1.9 (DIN)
- new net: D7.1 (K), R16.2
- new net: D7.2 (A), U1.20 (13_SCK_CRX1_LED)
- new net: R4.1, RV4.1, U3.7
- new net: RV2.1, U2.6 (-), U2.7
- new net: C8.1, RV2.2
- new net: R3.1, U3.1, U5.5 (+)
- new net: RV3.1, U5.6 (-), U5.7
- new net: C5.1, D1.1 (K), D2.2 (A), J1.T
- new net: R5.2, R9.2, U3.5 (+)
- new net: C6.1, D3.1 (K), D4.2 (A), J2.T
- new net: C23.2, RV4.2
- new net: R10.1, R3.2, U3.2 (-)
- new net: C24.1, R13.2, R15.1
- new net: RV5.2, U1.21 (14_A0_TX3_SPDIF_OUT)
- new net: C6.2, U2.5 (+)
- new net: C19.2, RV3.2
- new net: U5.1, U5.2 (-)
- new net +12V: C16.2, C18.2, C3.2, C34.2, C36.2, C4.2, D1.2 (A), D3.2 (A), J5.13 (Pin_13), J5.5 (Pin_5), R18.1, SW1.4, U2.4 (V-), U3.8 (V+), U5.4 (V-), VM4220M1.21 (VA)
- new net +5V: C29.1, C30.1, J5.14 (Pin_14), J5.6 (Pin_6), U1.33 (VIN)
- new net -12V: C1.1, C15.1, C17.1, C2.1, C33.1, C35.1, D2.1 (K), D4.1 (K), J5.1 (Pin_1), J5.9 (Pin_9), SW1.2, U2.8 (V+), U3.4 (V-), U5.8 (V+)
- new net GND1: C1.2, C10.2, C11.2, C12.2, C13.2, C14.2, C15.2, C16.1, C17.2, C18.1, C2.2, C20.2, C21.2, C22.2, C24.2, C25.2, C26.2, C3.1, C31.2, C32.2, C33.2, C34.1, C35.2, C36.1, C4.1, C9.2, FB1.1, J1.S, J2.S, J3.S, J4.S, J5.10 (Pin_10), J5.11 (Pin_11), J5.12 (Pin_12), J5.2 (Pin_2), J5.3 (Pin_3), J5.4 (Pin_4), R11.1, R12.2, R5.1, R6.1, RV1.3, RV2.3, RV3.3, RV4.3, U5.3 (+), VM4220M1.18 (DEM1), VM4220M1.22 (AGND)
- new net GND2: C27.2, C28.2, C29.2, C30.2, FB1.2, R16.1, RV5.1, U1.1 (GND), U1.32 (GND), VM4220M1.10 (DIF1), VM4220M1.11 (DIF0), VM4220M1.12 (DEM0), VM4220M1.7 (DGND)
- no-connect marks 0 -> 48
